File: hardware/esc/esc_module.kicad_sch (KiCad schematic)
At the start: 33 parts, among them J4 PHASE_A, J5 PHASE_B, J6 PHASE_C, U1 DRV8300DRGER, U2 STM32G071K8U6, U3 INA180A1

Commit message: h/feat: power stage
Connections:
- net SNS_BAT: no longer names the net of U2.13 (PA6)
- no-connect marks 15 -> 16
Changed lines of the file:
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@@
+	)
+	(no_connect
+		(at 184.15 66.04)
 	)
 	(no_connect
@@
 		(pts
 			(xy 85.09 73.66) (xy 87.63 73.66)
-		)
-		(stroke
-			(width 0)
-			(type default)
-		)
-	)
-	(wire
-		(pts
-			(xy 175.26 66.04) (xy 184.15 66.04)
 		)
 		(stroke
@@
 			)
 		)
-	)
-	(global_label "SNS_BAT"
-		(shape input)
-		(at 175.26 66.04 180)
-		(fields_autoplaced yes)
-		(effects
-			(font
-				(size 1.27 1.27)
-			)
-			(justify right)
-		)
-		(property "Intersheetrefs" "${INTERSHEET_REFS}"
-			(at 164.2315 66.04 0)
-			(hide yes)
-			(show_name no)
-			(do_not_autoplace no)
-			(effects
-				(font
-					(size 1.27 1.27)
-				)
-				(justify right)
-			)
-		)

Commit message: h/feat: placement; power stage pending
Parts:
- C4, C5, C8: value 0.1uF -> 1uF
- C7: footprint Capacitor_SMD:C_0805_2012Metric -> Capacitor_SMD:C_1206_3216Metric
Changed lines of the file:
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@@
 			)
 		)
-		(property "Value" "0.1uF"
+		(property "Value" "1uF"
 			(at 97.79 64.77 0)
 			(show_name no)
@@
 			)
 		)
-		(property "Value" "0.1uF"
+		(property "Value" "1uF"
 			(at 97.79 52.07 0)
 			(show_name no)
@@
 			)
 		)
-		(property "Footprint" "Capacitor_SMD:C_0805_2012Metric"
+		(property "Footprint" "Capacitor_SMD:C_1206_3216Metric"
 			(at 140.97 57.15 0)
 			(hide yes)
@@
 			)
 		)
-		(property "Value" "0.1uF"
+		(property "Value" "1uF"
 			(at 97.79 39.37 0)
 			(show_name no)

Commit message: h/feat: rework power stage: power drv8300 from 10v; remove 5v FC passthrough
Connections:
- net V_FET: no longer C6.1, C7.1, U1.4 (GVDD)
- new net V_10V: C6.1, C7.1, U1.4 (GVDD)
Changed lines of the file:
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@@
+	)
+	(junction
+		(at 243.84 88.9)
+		(diameter 0)
+		(color 0 0 0 0)
+	)
+	(junction
+		(at 128.27 158.75)
+		(diameter 0)
+		(color 0 0 0 0)
 	)
 	(junction
@@
 	)
 	(junction
-		(at 243.84 88.9)
-		(diameter 0)
-		(color 0 0 0 0)
-	)
-	(junction
-		(at 128.27 158.75)
-		(diameter 0)
-		(color 0 0 0 0)
-	)
-	(junction
 		(at 247.65 39.37)
 		(diameter 0)
@@
 	(wire
 		(pts
-			(xy 40.64 35.56) (xy 49.53 35.56)
+			(xy 46.99 35.56) (xy 49.53 35.56)
 		)
 		(stroke
@@
 	(wire
 		(pts
-			(xy 123.19 52.07) (xy 129.54 52.07)
-		)
-		(stroke
-			(width 0)
-			(type default)
-		)
-	)
-	(wire
-		(pts
 			(xy 138.43 170.18) (xy 138.43 167.64)
 		)
@@
 	(wire
 		(pts
-			(xy 140.97 52.07) (xy 147.32 52.07)
-		)
-		(stroke
-			(width 0)
-			(type default)
-		)
-	)
-	(wire
-		(pts
 			(xy 118.11 175.26) (xy 128.27 175.26)
 		)
@@
 	(wire
 		(pts
+			(xy 127 52.07) (xy 129.54 52.07)
+		)
+		(stroke
+			(width 0)
+			(type default)
+		)
+	)
+	(wire
+		(pts
 			(xy 146.05 149.86) (xy 154.94 149.86)
 		)
@@
 	(wire
 		(pts
+			(xy 140.97 52.07) (xy 143.51 52.07)
+		)
+		(stroke
+			(width 0)
+			(type default)
+		)
+	)
+	(wire
+		(pts
 			(xy 273.05 125.73) (xy 279.4 125.73)
 		)
@@
 	(wire
 		(pts
+			(xy 140.97 52.07) (xy 140.97 54.61)
+		)
+		(stroke
+			(width 0)
+			(type default)
+		)
+	)
+	(wire
+		(pts
 			(xy 46.99 71.12) (xy 46.99 66.04)
 		)
@@
 		(pts
 			(xy 184.15 63.5) (xy 175.26 63.5)
-		)
-		(stroke
-			(width 0)
-			(type default)
-		)
-	)
-	(wire
-		(pts
-			(xy 140.97 52.07) (xy 140.97 54.61)
 		)
 		(stroke
@@
 		)
 	)
-	(label "V_FET"
-		(at 40.64 35.56 0)
-		(effects
-			(font
-				(size 1.27 1.27)
-			)
-			(justify left bottom)
-		)
-	)
 	(label "SHA"
 		(at 104.14 40.64 0)
@@
 		)
 	)
-	(label "V_FET"
-		(at 147.32 52.07 180)
-		(effects
-			(font
-				(size 1.27 1.27)
-			)
-			(justify right bottom)
-		)
-	)
 	(label "BEMF_B"
 		(at 128.27 147.32 90)
@@
 		)
 	)
-	(label "V_FET"
-		(at 123.19 52.07 0)
-		(effects
-			(font
-				(size 1.27 1.27)
-			)
-			(justify left bottom)
-		)
-	)
 	(label "HA"
 		(at 175.26 76.2 0)
@@
 			)
 			(justify left bottom)
+		)
+	)
+	(global_label "V_10V"
+		(shape input)
+		(at 143.51 52.07 0)
+		(fields_autoplaced yes)
+		(effects
+			(font
+				(size 1.27 1.27)
+			)
+			(justify left)
+		)
+		(property "Intersheetrefs" "${INTERSHEET_REFS}"
+			(at 152.059 52.07 0)
+			(hide yes)
+			(show_name no)
+			(do_not_autoplace no)
+			(effects
+				(font
+					(size 1.27 1.27)
+				)
+				(justify left)
+			)
 		)
 	)
@@
 		)
 	)
+	(global_label "V_10V"
+		(shape input)
+		(at 46.99 35.56 180)
+		(fields_autoplaced yes)
+		(effects
+			(font
+				(size 1.27 1.27)
+			)
+			(justify right)
+		)
+		(property "Intersheetrefs" "${INTERSHEET_REFS}"
+			(at 38.441 35.56 0)
+			(hide yes)
+			(show_name no)
+			(do_not_autoplace no)
+			(effects
+				(font
+					(size 1.27 1.27)
+				)
+				(justify right)
+			)
+		)
+	)
 	(global_label "V_3V3"
 		(shape input)
@@
 			(hide yes)
 			(show_name no)
+			(do_not_autoplace no)
+			(effects
+				(font
+					(size 1.27 1.27)
+				)
+				(justify right)
+			)
+		)
+	)
+	(global_label "V_10V"
+		(shape input)
+		(at 127 52.07 180)
+		(fields_autoplaced yes)
+		(effects
+			(font
+				(size 1.27 1.27)
+			)
+			(justify right)
+		)
+		(property "Intersheetrefs" "${INTERSHEET_REFS}"
+			(at 118.451 52.07 0)
+			(hide yes)
+			(show_name no)
