File: hardware/esc/esc_module.kicad_sch (KiCad schematic)
At the start: 32 parts, among them J4 PHASE_A, J5 PHASE_B, J6 PHASE_C, U1 DRV8300DRGER, U15 ACS711xEXLT-31AB, U2 STM32G071K(8/B)U6

Commit message: h: final changes before fab
Parts:
- U2: LCSC# C529350 -> C724239; MPN STM32G071KBU6 -> STM32G071KBU3
Changed lines of the file:
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@@
 			)
 		)
-		(property "LCSC#" "C529350"
+		(property "LCSC#" "C724239"
 			(at 184.15 48.26 0)
 			(hide yes)
@@
 			)
 		)
-		(property "MPN" "STM32G071KBU6"
+		(property "MPN" "STM32G071KBU3"
 			(at 184.15 48.26 0)
 			(hide yes)
