File: hardware/esc/esc.kicad_pcb (KiCad board)
At the start: 8 copper layers, 38 x 41.5 mm, 219 parts, among them J1 TO_FC, J10 PHASE_A, J11 PHASE_B, J12 PHASE_C, J13 PHASE_A, J14 PHASE_B, J15 PHASE_C, J2 BAT_IN, J3 BAT_GND, J4 PHASE_A, J5 PHASE_B, J6 PHASE_C, J7 PHASE_A, J8 PHASE_B, J9 PHASE_C, Q1 NVTFWS003N04XMTAG, Q10 NVTFWS003N04XMTAG, Q11 NVTFWS003N04XMTAG, Q12 NVTFWS003N04XMTAG, Q13 NVTFWS003N04XMTAG, Q14 NVTFWS003N04XMTAG, Q15 NVTFWS003N04XMTAG, Q16 NVTFWS003N04XMTAG, Q17 NVTFWS003N04XMTAG, Q18 NVTFWS003N04XMTAG, Q19 NVTFWS003N04XMTAG, Q2 NVTFWS003N04XMTAG, Q20 NVTFWS003N04XMTAG, Q21 NVTFWS003N04XMTAG, Q22 NVTFWS003N04XMTAG, Q23 NVTFWS003N04XMTAG, Q24 NVTFWS003N04XMTAG, Q3 NVTFWS003N04XMTAG, Q4 NVTFWS003N04XMTAG, Q5 NVTFWS003N04XMTAG, Q6 NVTFWS003N04XMTAG, Q7 NVTFWS003N04XMTAG, Q8 NVTFWS003N04XMTAG, Q9 NVTFWS003N04XMTAG, U1 DRV8300DRGER, U10 DRV8300DRGER, U11 STM32G071K8U6, U12 INA180A1, U13 LMR51420YFDDCR, U14 LDLPUR212, U2 STM32G071K8U6, U3 INA180A1, U4 DRV8300DRGER, U5 STM32G071K8U6, U6 INA180A1, U7 DRV8300DRGER, U8 STM32G071K8U6, U9 INA180A1

Commit message: chore: nitpicky power trace
Routing:
- net /ESC Module 4/VIRTUAL: track 18.9 -> 20.5 mm
Changed lines of the file:
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@@
+	)
+	(segment
+		(start 156.239178 91.289178)
+		(end 155.72 90.77)
+		(width 0.6)
+		(layer "In4.Cu")
+		(net "V_10V")
+	)
+	(segment
+		(start 178.35 93.665286)
+		(end 178.35 93)
+		(width 0.6)
+		(layer "In4.Cu")
+		(net "V_10V")
+	)
+	(segment
+		(start 163.358614 98.63)
+		(end 159.947428 95.218814)
+		(width 0.6)
+		(layer "In4.Cu")
+		(net "V_10V")
+	)
+	(segment
+		(start 178.35 93)
+		(end 178.35 92.55)
+		(width 0.6)
+		(layer "In4.Cu")
+		(net "V_10V")
+	)
+	(segment
+		(start 159.947428 95.218814)
+		(end 159.947428 94.887428)
+		(width 0.6)
+		(layer "In4.Cu")
+		(net "V_10V")
+	)
+	(segment
+		(start 159.947428 94.887428)
+		(end 158.137818 93.077818)
+		(width 0.6)
+		(layer "In4.Cu")
+		(net "V_10V")
+	)
+	(segment
+		(start 171.52 102.07)
+		(end 172.013381 102.07)
+		(width 0.6)
+		(layer "In4.Cu")
+		(net "V_10V")
+	)
+	(segment
+		(start 170.02 99.036619)
+		(end 171.656619 97.4)
+		(width 0.6)
+		(layer "In4.Cu")
+		(net "V_10V")
+	)
+	(segment
+		(start 154.466081 87.680972)
+		(end 154.466081 87.22)
+		(width 0.6)
+		(layer "In4.Cu")
+		(net "V_10V")
+	)
+	(segment
+		(start 171.656619 97.4)
+		(end 172.313381 97.4)
+		(width 0.6)
+		(layer "In4.Cu")
+		(net "V_10V")
+	)
+	(segment
+		(start 175.924999 87.985001)
+		(end 176.974688 86.935312)
+		(width 0.6)
+		(layer "In4.Cu")
+		(net "V_10V")
+	)
+	(segment
+		(start 170.02 105.64)
+		(end 170.02 103.743381)
+		(width 0.6)
+		(layer "In4.Cu")
+		(net "V_10V")
+	)
+	(segment
+		(start 172.313381 97.4)
+		(end 175.924999 93.788382)
+		(width 0.6)
+		(layer "In4.Cu")
+		(net "V_10V")
+	)
+	(segment
+		(start 170.02 103.57)
+		(end 171.52 102.07)
+		(width 0.6)
+		(layer "In4.Cu")
+		(net "V_10V")
+	)
+	(segment
+		(start 172.013381 102.07)
+		(end 177.34338 96.740001)
+		(width 0.6)
+		(layer "In4.Cu")
+		(net "V_10V")
+	)
+	(segment
+		(start 170.02 103.743381)
+		(end 167.438309 101.161691)
+		(width 0.6)
+		(layer "In4.Cu")
+		(net "V_10V")
+	)
+	(segment
+		(start 156.239178 91.645377)
+		(end 156.239178 91.289178)
+		(width 0.6)
+		(layer "In4.Cu")
+		(net "V_10V")
+	)
+	(segment
+		(start 167.137748 100.861129)
+		(end 167.137748 100.457748)
+		(width 0.6)
+		(layer "In4.Cu")
+		(net "V_10V")
+	)
+	(segment
+		(start 176.974688 83.407698)
+		(end 177.642386 82.74)
+		(width 0.6)
+		(layer "In4.Cu")
+		(net "V_10V")
+	)
+	(segment
+		(start 166.895 108.765)
+		(end 158.83282 108.765)
+		(width 0.25)
+		(layer "In4.Cu")
+		(net "V_10V")
+	)
+	(segment
+		(start 165.31 98.63)
+		(end 163.358614 98.63)
+		(width 0.6)
+		(layer "In4.Cu")
+		(net "V_10V")
+	)
+	(segment
+		(start 177.642386 82.74)
+		(end 178.12 82.74)
+		(width 0.6)
+		(layer "In4.Cu")
+		(net "V_10V")
+	)
+	(segment
+		(start 176.974688 86.935312)
+		(end 176.974688 83.407698)
+		(width 0.6)
+		(layer "In4.Cu")
+		(net "V_10V")
 	)
 	(segment
@@
 	)
 	(segment
+		(start 155.081129 100.861129)
+		(end 154.46 100.24)
+		(width 0.6)
+		(layer "In4.Cu")
+		(net "V_10V")
+	)
+	(segment
+		(start 170.02 105.64)
+		(end 166.895 108.765)
+		(width 0.25)
+		(layer "In4.Cu")
+		(net "V_10V")
+	)
+	(segment
+		(start 167.438309 101.161691)
+		(end 167.137748 100.861129)
+		(width 0.6)
+		(layer "In4.Cu")
+		(net "V_10V")
+	)
+	(segment
+		(start 154.466081 89.899462)
+		(end 154.466081 87.680972)
+		(width 0.6)
+		(layer "In4.Cu")
+		(net "V_10V")
+	)
+	(segment
+		(start 158.83282 108.765)
+		(end 158.642832 108.575012)
+		(width 0.25)
+		(layer "In4.Cu")
+		(net "V_10V")
+	)
+	(segment
 		(start 155.336619 90.77)
 		(end 154.466081 89.899462)
@@
 	)
 	(segment
-		(start 178.35 93.665286)
-		(end 178.35 93)
-		(width 0.6)
-		(layer "In4.Cu")
-		(net "V_10V")
-	)
-	(segment
-		(start 178.35 93)
-		(end 178.35 92.55)
-		(width 0.6)
-		(layer "In4.Cu")
-		(net "V_10V")
-	)
-	(segment
-		(start 159.947428 94.887428)
-		(end 158.137818 93.077818)
-		(width 0.6)
-		(layer "In4.Cu")
-		(net "V_10V")
-	)
-	(segment
-		(start 171.52 102.07)
-		(end 172.013381 102.07)
-		(width 0.6)
-		(layer "In4.Cu")
-		(net "V_10V")
-	)
-	(segment
-		(start 170.02 99.036619)
-		(end 171.656619 97.4)
-		(width 0.6)
-		(layer "In4.Cu")
-		(net "V_10V")
-	)
-	(segment
-		(start 154.466081 87.680972)
-		(end 154.466081 87.22)
-		(width 0.6)
-		(layer "In4.Cu")
-		(net "V_10V")
-	)
-	(segment
-		(start 171.656619 97.4)
-		(end 172.313381 97.4)
-		(width 0.6)
-		(layer "In4.Cu")
-		(net "V_10V")
-	)
-	(segment
-		(start 175.924999 87.985001)
-		(end 176.974688 86.935312)
-		(width 0.6)
-		(layer "In4.Cu")
-		(net "V_10V")
-	)
-	(segment
-		(start 170.02 105.64)
-		(end 170.02 103.743381)
-		(width 0.6)
-		(layer "In4.Cu")
-		(net "V_10V")
-	)
-	(segment
-		(start 172.313381 97.4)
-		(end 175.924999 93.788382)
+		(start 178.48 82.07)
+		(end 178.48 81.6)
 		(width 0.6)
 		(layer "In4.Cu")
@@
 	)
 	(segment
-		(start 170.02 103.57)
-		(end 171.52 102.07)
-		(width 0.6)
-		(layer "In4.Cu")
-		(net "V_10V")
-	)
-	(segment
-		(start 172.013381 102.07)
-		(end 177.34338 96.740001)
-		(width 0.6)
-		(layer "In4.Cu")
-		(net "V_10V")
-	)
-	(segment
-		(start 170.02 103.743381)
-		(end 167.438309 101.161691)
-		(width 0.6)
-		(layer "In4.Cu")
-		(net "V_10V")
-	)
-	(segment
-		(start 159.947428 95.218814)
-		(end 159.947428 94.887428)
-		(width 0.6)
-		(layer "In4.Cu")
-		(net "V_10V")
-	)
-	(segment
-		(start 165.890305 101.161691)
-		(end 159.947428 95.218814)
-		(width 0.6)
-		(layer "In4.Cu")
-		(net "V_10V")
-	)
-	(segment
-		(start 156.239178 91.289178)
-		(end 155.72 90.77)
-		(width 0.6)
-		(layer "In4.Cu")
-		(net "V_10V")
-	)
-	(segment
-		(start 176.974688 83.407698)
-		(end 177.642386 82.74)
-		(width 0.6)
-		(layer "In4.Cu")
-		(net "V_10V")
-	)
-	(segment
-		(start 166.895 108.765)
-		(end 158.83282 108.765)
-		(width 0.25)
-		(layer "In4.Cu")
-		(net "V_10V")
-	)
-	(segment
-		(start 154.466081 89.899462)
-		(end 154.466081 87.680972)
-		(width 0.6)
-		(layer "In4.Cu")
-		(net "V_10V")
-	)
-	(segment
-		(start 177.642386 82.74)
-		(end 178.12 82.74)
-		(width 0.6)
-		(layer "In4.Cu")
-		(net "V_10V")
-	)
-	(segment
-		(start 176.974688 86.935312)
-		(end 176.974688 83.407698)
-		(width 0.6)
-		(layer "In4.Cu")
-		(net "V_10V")
-	)
-	(segment
-		(start 155.081129 100.861129)
-		(end 154.46 100.24)
-		(width 0.6)
-		(layer "In4.Cu")
-		(net "V_10V")
-	)
-	(segment
-		(start 170.02 105.64)
-		(end 166.895 108.765)
-		(width 0.25)
-		(layer "In4.Cu")
-		(net "V_10V")
-	)
-	(segment
-		(start 167.438309 101.161691)
-		(end 167.137748 100.861129)
-		(width 0.6)
-		(layer "In4.Cu")
-		(net "V_10V")
-	)
-	(segment
-		(start 158.83282 108.765)
-		(end 158.642832 108.575012)
-		(width 0.25)
-		(layer "In4.Cu")
-		(net "V_10V")
-	)
-	(segment
-		(start 178.48 82.07)
-		(end 178.48 81.6)
-		(width 0.6)
-		(layer "In4.Cu")
-		(net "V_10V")
-	)
-	(segment
 		(start 178.12 82.74)
 		(end 178.48 82.38)
@@
 	(segment
 		(start 167.137748 100.861129)
-		(end 155.081129 100.861129)
+		(end 166.82 100.861129)
 		(width 0.6)
 		(layer "In4.Cu")
@@
 	)
 	(segment
-		(start 167.438309 101.161691)
-		(end 165.890305 101.161691)
-		(width 0.6)
-		(layer "In4.Cu")
-		(net "V_10V")
-	)
-	(segment
 		(start 170.02 105.64)
 		(end 170.02 103.57)
@@
 	)
 	(segment
+		(start 166.82 100.861129)
+		(end 155.081129 100.861129)
+		(width 0.6)
+		(layer "In4.Cu")
+		(net "V_10V")
+	)
+	(segment
 		(start 154.46 100.24)
 		(end 154.46 99.782947)
@@
 	)
 	(segment
-		(start 156.239178 91.645377)
-		(end 156.239178 91.289178)
+		(start 167.137748 100.457748)
+		(end 165.31 98.63)
 		(width 0.6)
 		(layer "In4.Cu")
@@
 		(net "/ESC Module 4/VIRTUAL")
 	)
+	(segment
+		(start 167.438309 101.161691)
+		(end 168.986313 101.161691)
+		(width 0.6)
+		(layer "In3.Cu")
+		(net "/ESC Module 4/VIRTUAL")
+	)

Commit message: h/feat: silkscreen
Parts:
- added G***: LOGO, Stratus:Logo, B.Cu at (178.2, 104.0)
Routing:
- net /ESC Module 4/VIRTUAL: track 20.5 -> 18.9 mm
- net /ESC Module 1/PHASE_C: track 18.9 -> 20.0 mm
Other:
- board text added: "GND"
- board text added: "Jett"
- board text added: "M1"
- board text added: "M2"
- board text added: "M4"
- board text added: "Rev. 2"
- board text added: "TELEM"
- board text added: "VBAT"

Commit message: h/fix: add missing silkscreen
Other:
- board text added: "M3"
Changed lines of the file:
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@@
+		)
+	)
+	(gr_text "M3"
+		(at 169.037956 76.95 270)
+		(layer "B.SilkS" knockout)
+		(effects
+			(font
+				(face "OCR-A BT")
+				(size 0.75 0.75)
+			)
+			(justify left bottom mirror)
+		)
+		(render_cache "M3" 270
+			(polygon
+				(pts
+					(xy 169.801464 76.842838) (xy 169.801464 76.733616) (xy 169.648186 76.625447) (xy 169.801464 76.517278)
+					(xy 169.801464 76.408101) (xy 169.170676 76.408101) (xy 169.150344 76.411329) (xy 169.135093 76.42042)
+					(xy 169.124946 76.434365) (xy 169.121492 76.452156) (xy 169.124996 76.469976) (xy 169.135322 76.483984)
+					(xy 169.150732 76.493068) (xy 169.170676 76.496257) (xy 169.67635 76.496257) (xy 169.558977 76.581391)
+					(xy 169.540017 76.581391) (xy 169.519638 76.58462) (xy 169.504342 76.59371) (xy 169.494231 76.607652)
+					(xy 169.490787 76.625447) (xy 169.494292 76.643266) (xy 169.504617 76.657274) (xy 169.520065 76.66636)
+					(xy 169.540017 76.669548) (xy 169.558977 76.669548) (xy 169.67635 76.754682) (xy 169.170676 76.754682)
+					(xy 169.150344 76.75791) (xy 169.135093 76.767001) (xy 169.124946 76.780946) (xy 169.121492 76.798737)
+					(xy 169.124996 76.816556) (xy 169.135322 76.830565) (xy 169.150732 76.839649) (xy 169.170676 76.842838)
+				)
+			)
+			(polygon
+				(pts
+					(xy 169.801464 76.145143) (xy 169.801464 75.847793) (xy 169.798586 75.824935) (xy 169.790098 75.804491)
+					(xy 169.775635 75.785785) (xy 169.757125 75.771168) (xy 169.736663 75.762565) (xy 169.713536 75.759636)
+					(xy 169.549634 75.759636) (xy 169.526937 75.761687) (xy 169.505029 75.767834) (xy 169.48402 75.777856)
+					(xy 169.462485 75.792426) (xy 169.439496 75.777864) (xy 169.417194 75.767834) (xy 169.394295 75.76165)
+					(xy 169.371902 75.759636) (xy 169.209419 75.759636) (xy 169.186275 75.762539) (xy 169.165812 75.771058)
+					(xy 169.14732 75.785511) (xy 169.132897 75.804057) (xy 169.12439 75.824581) (xy 169.121492 75.847793)
+					(xy 169.121492 76.145143) (xy 169.124709 76.165526) (xy 169.133765 76.180818) (xy 169.1477 76.190931)
+					(xy 169.165456 76.194373) (xy 169.183188 76.190871) (xy 169.197146 76.180543) (xy 169.206232 76.165095)
+					(xy 169.209419 76.145143) (xy 169.209419 75.848846) (xy 169.373413 75.848846) (xy 169.389698 75.852053)
+					(xy 169.404188 75.861898) (xy 169.414215 75.876251) (xy 169.417514 75.892901) (xy 169.417514 76.059047)
+					(xy 169.420647 76.079747) (xy 169.429238 76.094402) (xy 169.442841 76.103881) (xy 169.461478 76.107224)
+					(xy 169.478859 76.103863) (xy 169.492894 76.093898) (xy 169.502172 76.078886) (xy 169.505442 76.059047)
+					(xy 169.505442 75.892901) (xy 169.508691 75.876234) (xy 169.518539 75.861898) (xy 169.532916 75.852086)
+					(xy 169.549634 75.848846) (xy 169.713536 75.848846) (xy 169.713536 76.145143) (xy 169.716718 76.165942)
+					(xy 169.725535 76.181047) (xy 169.739332 76.190951) (xy 169.7575 76.194373) (xy 169.775233 76.190871)
+					(xy 169.789191 76.180543) (xy 169.798276 76.165095)
+				)
+			)
 		)
 	)

Commit message: h/fix: add polarity indicators
Other:
- board text added: "+"
- board text added: "-"
Changed lines of the file:
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@@
+	)
+	(gr_circle
+		(center 151.15 76.342706)
+		(end 152.9 76.342706)
+		(stroke
+			(width 0.25)
+			(type dash)
+		)
+		(fill no)
+		(layer "F.SilkS")
+	)
+	(gr_circle
+		(center 151.15 106.857671)
+		(end 152.9 106.857671)
+		(stroke
+			(width 0.25)
+			(type dash)
+		)
+		(fill no)
+		(layer "F.SilkS")
+	)
+	(gr_circle
+		(center 181.700754 76.342706)
+		(end 183.450754 76.342706)
+		(stroke
+			(width 0.25)
+			(type dash)
+		)
+		(fill no)
+		(layer "F.SilkS")
+	)
+	(gr_circle
+		(center 181.700754 106.847633)
+		(end 183.450754 106.847633)
+		(stroke
+			(width 0.25)
+			(type dash)
+		)
+		(fill no)
+		(layer "F.SilkS")
 	)
 	(gr_circle
@@
 		(layer "Edge.Cuts")
 	)
+	(gr_text "+"
+		(at 160.81 108.53 0)
+		(layer "F.SilkS")
+		(effects
+			(font
+				(size 1.25 1.25)
+			)
+			(justify left bottom)
+		)
+	)
+	(gr_text "-"
+		(at 170.31 108.53 0)
+		(layer "F.SilkS")
+		(effects
+			(font
+				(size 1.25 1.25)
+			)
+			(justify left bottom)
+		)
+	)
 	(gr_text "VBAT"
