File: hardware/esc/esc.kicad_sch (KiCad schematic)
At the start: 12 parts, among them J1 TO_FC, J2 BAT_IN, J3 BAT_GND

Commit message: chore: add BOM
Parts:
- D1, D2: LCSC# (none) -> C3000897; MFR (none) -> Vishay; MPN (none) -> VLMTG1400-GS08; Manufacturer_Name Vishay -> (none); Manufacturer_Part_Number VLMTG1500-GS08 -> (none)
- D3: LCSC# (none) -> C148209; MFR (none) -> Littelfuse; MPN (none) -> SMAJ20A
- J1: LCSC# (none) -> C160408; MFR (none) -> JST; MPN (none) -> SM09B-SRSS-TB(LF)(SN); Manufacturer_Name JST -> (none); Manufacturer_Part_Number SM09B-SRSS-TB -> (none)
- R1, R3: LCSC# (none) -> C106235; MFR (none) -> Yageo; MPN (none) -> RC0402FR-071KL; Manufacturer_Name Yageo -> (none); Manufacturer_Part_Number RC0402FR-071KL -> (none)
Other:
- title: 2S LiHV 4-in-1 BLDC ESC -> 2-4S 4-in-1 BLDC ESC
Changed lines of the file:
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@@
 	(paper "A4")
 	(title_block
-		(title "2S LiHV 4-in-1 BLDC ESC")
-		(date "2026-07-06")
-		(rev "A")
+		(title "2-4S 4-in-1 BLDC ESC")
+		(date "2026-09-10")
+		(rev "2")
 		(company "Stratus")
-		(comment 1 "Passives >= 2.2uF -> 0603")
-		(comment 2 "Passives >= 10uF -> 0805")
-		(comment 3 "Target rating: ~20A continuous per motor, ~80A total continuous")
-		(comment 4 "This board placed below FC")
+		(comment 1 "Caps on 10/5V rails: 16V+; VBAT: 30V+")
+		(comment 2 "~20A continuous per motor, ~80A total continuous")
+		(comment 3 "This board placed below FC")
 	)
 	(rectangle
@@
 			)
 		)
-		(property "Description" "Generic connector, single row, 01x01, script generated (kicad-library-utils/schlib/autogen/connector/)"
+		(property "Description" "Battery input pad"
+			(at 161.29 151.13 0)
+			(hide yes)
+			(show_name no)
+			(do_not_autoplace no)
+			(effects
+				(font
+					(size 1.27 1.27)
+				)
+			)
+		)
+		(property "LCSC#" ""
 			(at 161.29 151.13 0)
 			(hide yes)
@@
 			)
 		)
-		(property "Description" "Light emitting diode, small symbol"
+		(property "Description" "0603 Green LED"
 			(at 120.65 123.19 0)
 			(hide yes)
@@
 			)
 		)
-		(property "Manufacturer_Name" "Vishay"
+		(property "LCSC#" "C3000897"
 			(at 120.65 123.19 0)
 			(hide yes)
@@
 			)
 		)
-		(property "Manufacturer_Part_Number" "VLMTG1500-GS08"
+		(property "MFR" "Vishay"
+			(at 120.65 123.19 0)
+			(hide yes)
+			(show_name no)
+			(do_not_autoplace no)
+			(effects
+				(font
+					(size 1.27 1.27)
+				)
+			)
+		)
+		(property "MPN" "VLMTG1400-GS08"
 			(at 120.65 123.19 0)
 			(hide yes)
@@
 			)
 		)
-		(property "Description" "Resistor, small symbol"
+		(property "Description" "0402 1k"
 			(at 128.27 133.35 0)
 			(hide yes)
@@
 			)
 		)
-		(property "Manufacturer_Name" "Yageo"
+		(property "LCSC#" "C106235"
 			(at 128.27 133.35 90)
 			(hide yes)
@@
 			)
 		)
-		(property "Manufacturer_Part_Number" "RC0402FR-071KL"
+		(property "MFR" "Yageo"
+			(at 128.27 133.35 90)
+			(hide yes)
+			(show_name no)
+			(do_not_autoplace no)
+			(effects
+				(font
+					(size 1.27 1.27)
+				)
+			)
+		)
+		(property "MPN" "RC0402FR-071KL"
 			(at 128.27 133.35 90)
 			(hide yes)
@@
 			)
 		)
-		(property "Description" "Light emitting diode, small symbol"
+		(property "Description" "0603 Green LED"
 			(at 120.65 133.35 0)
 			(hide yes)
@@
 			)
 		)
-		(property "Manufacturer_Name" "Vishay"
+		(property "LCSC#" "C3000897"
 			(at 120.65 133.35 0)
 			(hide yes)
@@
 			)
 		)
-		(property "Manufacturer_Part_Number" "VLMTG1500-GS08"
+		(property "MFR" "Vishay"
+			(at 120.65 133.35 0)
+			(hide yes)
+			(show_name no)
+			(do_not_autoplace no)
+			(effects
+				(font
+					(size 1.27 1.27)
+				)
+			)
+		)
+		(property "MPN" "VLMTG1400-GS08"
 			(at 120.65 133.35 0)
 			(hide yes)
@@
 			)
 		)
-		(property "Description" "Generic connector, single row, 01x01, script generated (kicad-library-utils/schlib/autogen/connector/)"
+		(property "Description" "Battery input pad"
+			(at 161.29 144.78 0)
+			(hide yes)
+			(show_name no)
+			(do_not_autoplace no)
+			(effects
+				(font
+					(size 1.27 1.27)
+				)
+			)
+		)
+		(property "LCSC#" ""
 			(at 161.29 144.78 0)
 			(hide yes)
@@
 			)
 		)
-		(property "Description" "400W unidirectional Transient Voltage Suppressor, 20.0Vr, SMA(DO-214AC)"
+		(property "Description" "32.4VC DO-214AC"
+			(at 128.27 157.48 0)
+			(hide yes)
+			(show_name no)
+			(do_not_autoplace no)
+			(effects
+				(font
+					(size 1.27 1.27)
+				)
+			)
+		)
+		(property "LCSC#" "C148209"
+			(at 128.27 157.48 0)
+			(hide yes)
+			(show_name no)
+			(do_not_autoplace no)
+			(effects
+				(font
+					(size 1.27 1.27)
+				)
+			)
+		)
+		(property "MFR" "Littelfuse"
+			(at 128.27 157.48 0)
+			(hide yes)
+			(show_name no)
+			(do_not_autoplace no)
+			(effects
+				(font
+					(size 1.27 1.27)
+				)
+			)
+		)
+		(property "MPN" "SMAJ20A"
 			(at 128.27 157.48 0)
 			(hide yes)
@@
 			)
 		)
+		(property "LCSC#" ""
+			(at 186.69 109.22 0)
+			(hide yes)
+			(show_name no)
+			(do_not_autoplace no)
+			(effects
+				(font
+					(size 1.27 1.27)
+				)
+			)
+		)
 		(instances
 			(project "esc"
@@
 			)
 		)
-		(property "Description" "Resistor, small symbol"
+		(property "Description" "0402 1k"
 			(at 128.27 123.19 0)
 			(hide yes)
@@
 			)
 		)
-		(property "Manufacturer_Name" "Yageo"
+		(property "LCSC#" "C106235"
 			(at 128.27 123.19 90)
 			(hide yes)
@@
 			)
 		)
-		(property "Manufacturer_Part_Number" "RC0402FR-071KL"
+		(property "MFR" "Yageo"
+			(at 128.27 123.19 90)
+			(hide yes)
+			(show_name no)
+			(do_not_autoplace no)
+			(effects
+				(font
+					(size 1.27 1.27)
+				)
+			)
+		)
+		(property "MPN" "RC0402FR-071KL"
 			(at 128.27 123.19 90)
 			(hide yes)
@@
 			)
 		)
+		(property "LCSC#" ""
+			(at 199.39 118.11 0)
+			(hide yes)
+			(show_name no)
+			(do_not_autoplace no)
+			(effects
+				(font
+					(size 1.27 1.27)
+				)
+			)
+		)
 		(instances
 			(project "esc"
@@
 			)
 		)
+		(property "LCSC#" ""
+			(at 186.69 118.11 0)
+			(hide yes)
+			(show_name no)
+			(do_not_autoplace no)
+			(effects
+				(font
+					(size 1.27 1.27)
+				)
+			)
+		)
 		(instances
 			(project "esc"
@@
 			)
 		)
-		(property "Description" "Generic connector, single row, 01x09, script generated (kicad-library-utils/schlib/autogen/connector/)"
+		(property "Description" "Horizontal JST-SH 1x9"
 			(at 158.75 127 0)
 			(hide yes)
@@
 			)
 		)
-		(property "Manufacturer_Name" "JST"
+		(property "LCSC#" "C160408"
 			(at 158.75 127 0)
 			(hide yes)
@@
 			)
 		)
-		(property "Manufacturer_Part_Number" "SM09B-SRSS-TB"
+		(property "MFR" "JST"
+			(at 158.75 127 0)
+			(hide yes)
+			(show_name no)
+			(do_not_autoplace no)
+			(effects
+				(font
+					(size 1.27 1.27)
+				)
+			)
+		)
+		(property "MPN" "SM09B-SRSS-TB(LF)(SN)"
 			(at 158.75 127 0)
 			(hide yes)
@@
 			(at 199.39 109.22 0)
 			(hide yes)
+			(show_name no)
+			(do_not_autoplace no)
+			(effects
+				(font
+					(size 1.27 1.27)
+				)
+			)
+		)
+		(property "LCSC#" ""
+			(at 199.39 109.22 0)
+			(hide yes)

Commit message: h: leds
Parts:
- R3: value 1k -> 10k
Changed lines of the file:
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@@
 			)
 		)
-		(property "Value" "1k"
+		(property "Value" "10k"
 			(at 128.27 130.81 90)
 			(show_name no)

Commit message: esc: rev 3, mainly visual changes
Parts:
- J1: footprint Connector_JST:JST_SH_SM09B-SRSS-TB_1x09-1MP_P1.00mm_Horizontal -> Stratus:JST_SH_1x9_ESC
Changed lines of the file:
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@@
 			)
 		)
-		(property "Footprint" "Connector_JST:JST_SH_SM09B-SRSS-TB_1x09-1MP_P1.00mm_Horizontal"
+		(property "Footprint" "Stratus:JST_SH_1x9_ESC"
 			(at 158.75 127 0)
 			(hide yes)

Commit message: h: prep for rev 3; layout, stackup changes
Parts:
- H1, H2, H3, H4: now fitted
- R3: LCSC# C106235 -> C60490; MPN RC0402FR-071KL -> RC0402FR-0710KL
Changed lines of the file:
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@@
 			)
 		)
-		(property "Description" "0402 1k"
+		(property "Description" "0402 10k"
 			(at 128.27 133.35 0)
 			(hide yes)
@@
 			)
 		)
-		(property "LCSC#" "C106235"
+		(property "LCSC#" "C60490"
 			(at 128.27 133.35 90)
 			(hide yes)
@@
 			)
 		)
-		(property "MPN" "RC0402FR-071KL"
+		(property "MPN" "RC0402FR-0710KL"
 			(at 128.27 133.35 90)
 			(hide yes)
@@
 		(on_board yes)
 		(in_pos_files yes)
-		(dnp yes)
+		(dnp no)
 		(fields_autoplaced yes)
 		(property "Reference" "H1"
@@
 		(on_board yes)
 		(in_pos_files yes)
-		(dnp yes)
+		(dnp no)
 		(fields_autoplaced yes)
 		(property "Reference" "H4"
@@
 		(on_board yes)
 		(in_pos_files yes)
-		(dnp yes)
+		(dnp no)
 		(fields_autoplaced yes)
 		(property "Reference" "H3"
@@
 		(on_board yes)
 		(in_pos_files yes)
-		(dnp yes)
+		(dnp no)
 		(fields_autoplaced yes)
 		(property "Reference" "H2"
