File: hardware/esc/esc.kicad_sch (KiCad schematic)
At the start: 12 parts, among them J1 TO_FC, J2 BAT_IN, J3 BAT_GND

Commit message: h: update BOM and FET for 5S
Parts:
- D3: value SMAJ20A -> SMAJ24A; LCSC# C148209 -> C148222; MPN SMAJ20A -> SMAJ24A
Changed lines of the file:
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@@
 			)
 		)
-		(property "Value" "SMAJ20A"
+		(property "Value" "SMAJ24A"
 			(at 179.07 43.18 0)
 			(show_name no)
@@
 			)
 		)
-		(property "Description" "32.4VC DO-214AC"
+		(property "Description" "38.9VC DO-214AC"
 			(at 179.07 46.99 0)
 			(hide yes)
@@
 			)
 		)
-		(property "LCSC#" "C148209"
+		(property "LCSC#" "C148222"
 			(at 179.07 46.99 0)
 			(hide yes)
@@
 			)
 		)
-		(property "MPN" "SMAJ20A"
+		(property "MPN" "SMAJ24A"
 			(at 179.07 46.99 0)
 			(hide yes)

Commit message: h: sync
Other:
- title: 2-4S 4-in-1 BLDC ESC -> 2-5S 4-in-1 BLDC ESC
Changed lines of the file:
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@@
 	(paper "A4")
 	(title_block
-		(title "2-4S 4-in-1 BLDC ESC")
-		(date "2026-09-10")
-		(rev "2")
+		(title "2-5S 4-in-1 BLDC ESC")
+		(date "2026-10-13")
+		(rev "3")
 		(company "Stratus")
 		(comment 1 "Caps on 10/5V rails: 16V+; VBAT: 30V+")
-		(comment 2 "~20A continuous per motor, ~80A total continuous")
+		(comment 2 "~25A continuous per motor, ~100A total continuous")
 		(comment 3 "This board placed below FC")
 	)

Commit message: general: update ESC schem and README
Parts:
- removed D1, D2: Green, LED_SMD:LED_0603_1608Metric, symbol Device:LED_Small
- removed D3: SMAJ24A, Stratus:SMAJ20A, symbol Diode:SMAJ20A
- removed R1: 1k, Stratus:R_0402, symbol Device:R_Small
- removed R3: 10k, Stratus:R_0402, symbol Device:R_Small
Other:
- note removed: "Indicators"
- note removed: "TVS"
- title: 2-5S 4-in-1 BLDC ESC -> 3-5S 4-in-1 BLDC ESC
- moved on the sheet: H1, H2, H3, H4, J1, J2, J3
