File: hardware/esc/power.kicad_sch (KiCad schematic)
At the start: 37 parts, among them U13 LMR51420YFDDCR, U14 LDLPUR212

Commit message: h/feat: clean up connections and DRC violations
Parts:
- R74: value 31.6k -> 18k
Changed lines of the file:
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@@
 			)
 		)
-		(property "Value" "31.6k"
+		(property "Value" "18k"
 			(at 226.06 57.1499 0)
 			(show_name no)

Commit message: chore: add BOM
Parts:
- C39: LCSC# (none) -> C343047; MFR (none) -> TDK; MPN (none) -> CGA2B3X7R1V104KT0Y0F; Manufacturer_Name Samsung -> (none); Manufacturer_Part_Number CL05A104KA5NNNC -> (none)
- C40, C69: value 10uF -> 4.7uF; LCSC# (none) -> C22385335; MFR (none) -> Taiyo Yuden; MPN (none) -> TDK105CBJ475MV-F; Manufacturer_Name Murata -> (none); Manufacturer_Part_Number GRM188R61E475KE11D -> (none)
- C42, C65, C68: value 10uF -> 4.7uF; LCSC# (none) -> C22385335; MFR (none) -> Taiyo Yuden; MPN (none) -> TDK105CBJ475MV-F; Manufacturer_Name Samsung -> (none); Manufacturer_Part_Number CL21A226MAYNNWE -> (none)
- C43: LCSC# (none) -> C3835721; MFR (none) -> Murata; MPN (none) -> GRM155R6YA105KE11J; Manufacturer_Name TDK -> (none); Manufacturer_Part_Number C1005X5R1E105K050BC -> (none)
- C44, C45, C46, C47, C48, C49, C50, C54, C55, C56, C57, C58: LCSC# (none) -> C162422; MFR (none) -> Murata; MPN (none) -> GRM21BR6YA106KE43L
- C51, C52, C53, C61, C62, C63, C71, C72: LCSC# (none) -> C162422; MFR (none) -> Murata; MPN (none) -> GRM21BR6YA106KE43L; Manufacturer_Name Samsung -> (none); Manufacturer_Part_Number CL21A226MAYNNWE -> (none)
- C66, C67: value 10uF -> 4.7uF; LCSC# (none) -> C307467; MFR (none) -> Samsung; MPN (none) -> CL10A475KL8NRNC; Manufacturer_Name Samsung -> (none); Manufacturer_Part_Number CL21A226MAYNNWE -> (none)
- C70: LCSC# (none) -> C343047; MFR (none) -> TDK; MPN (none) -> CGA2B3X7R1V104KT0Y0F; Manufacturer_Name TDK -> (none); Manufacturer_Part_Number C1005X5R1E105K050BC -> (none)
- L1: LCSC# (none) -> C3224690; MFR (none) -> TDK; MPN (none) -> BCL322520RT-4R7M-D; Manufacturer_Name Taiyo Yuden -> (none); Manufacturer_Part_Number MDWK4040T4R7MM -> (none)
- R74: LCSC# (none) -> C138044; MFR (none) -> Yageo; MPN (none) -> RC0402FR-0718KL; Manufacturer_Name Yageo -> (none); Manufacturer_Part_Number RC0402FR-0731K6L -> (none)
- R75: value 158k -> 160k; LCSC# (none) -> C273334; MFR (none) -> Yageo; MPN (none) -> RC0402FR-07160KL; Manufacturer_Name Yageo -> (none); Manufacturer_Part_Number RC0402FR-0756KL -> (none)
- R76, R77: LCSC# (none) -> C60490; MFR (none) -> Yageo; MPN (none) -> RC0402FR-0710KL; Manufacturer_Name Yageo -> (none); Manufacturer_Part_Number RC0402FR-0710KL -> (none)
- U13: LCSC# (none) -> C7296200; MFR (none) -> TI; MPN (none) -> LMR51420YFDDCR
- U14: value LDLPUR212 -> LDL212PUR; LCSC# (none) -> C2969849; MFR (none) -> ST; MPN (none) -> LDL212PUR; Manufacturer_Name onsemi -> (none); Manufacturer_Part_Number NCP59800BMNADJTAG -> (none)
Other:
- company: (none) -> Stratus
- title: (none) -> Power Stages

Commit message: h: prep for rev 3; layout, stackup changes
Parts:
- R75: LCSC# C273334 -> C226798; MPN RC0402FR-07160KL -> AC0402FR-07160KL
Changed lines of the file:
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@@
 			)
 		)
-		(property "LCSC#" "C273334"
+		(property "LCSC#" "C226798"
 			(at 113.03 59.69 0)
 			(hide yes)
@@
 			)
 		)
-		(property "MPN" "RC0402FR-07160KL"
+		(property "MPN" "AC0402FR-07160KL"
 			(at 113.03 59.69 0)
 			(hide yes)
