File: hardware/esc/half_bridge.kicad_sch (KiCad schematic)
At the start: 4 parts, among them Q1 AGM4025AP, Q2 AGM4025AP

Commit message: h: update FET footprint
Parts:
- Q1, Q2: footprint Stratus:CSD17575Q3 -> Stratus:AGM4025AP
Changed lines of the file:
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@@
 			)
 		)
-		(property "Footprint" "Stratus:CSD17575Q3"
+		(property "Footprint" "Stratus:AGM4025AP"
 			(at 148.59 207.95 0)
 			(hide yes)
@@
 			)
 		)
-		(property "Footprint" "Stratus:CSD17575Q3"
+		(property "Footprint" "Stratus:AGM4025AP"
 			(at 148.59 172.39 0)
 			(hide yes)
