File: hardware/fc/osd.kicad_sch (KiCad schematic)
At the start: 17 parts, among them U11 OPA354AIDBVR, U8 TS5A3159ADCK, U9 TLV7031DCKR

Commit message: fc: schematic footprint changes
Parts:
- U9: footprint Package_TO_SOT_SMD:SOT-353_SC-70-5 -> Package_TO_SOT_SMD:SOT-363_SC-70-6
Changed lines of the file:
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@@
 			)
 		)
-		(property "Footprint" "Package_TO_SOT_SMD:SOT-353_SC-70-5"
+		(property "Footprint" "Package_TO_SOT_SMD:SOT-363_SC-70-6"
 			(at 190.5 144.78 0)
 			(hide yes)
