File: hardware/fc/peripherals.kicad_sch (KiCad schematic)
At the start: 13 parts, among them J1 USB4110-GF-A, J2 Micro_SD_Card_Det1, J3 FROM_ESC, J4 CAM, J5 CAM_CC, J6 ELRS, J7 VTX, U4 USBLC6-2SC6, U5 EMIF06-MSD02N16

Commit message: fc: delete barometer; finalise schematic
Changed lines of the file:
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@@
 	)
 	(junction
-		(at 129.54 92.71)
+		(at 139.7 92.71)
 		(diameter 0)
 		(color 0 0 0 0)
@@
 	(wire
 		(pts
-			(xy 129.54 95.25) (xy 129.54 92.71)
+			(xy 139.7 95.25) (xy 139.7 92.71)
 		)
 		(stroke
@@
 	(symbol
 		(lib_id "power:GND")
-		(at 129.54 95.25 0)
+		(at 139.7 95.25 0)
 		(mirror y)
 		(unit 1)
@@
 		(dnp no)
 		(property "Reference" "#PWR033"
-			(at 129.54 101.6 0)
+			(at 139.7 101.6 0)
 			(hide yes)
 			(show_name no)
@@
 		)
 		(property "Value" "GND"
-			(at 125.476 97.282 0)
+			(at 135.636 97.282 0)
 			(show_name no)
 			(do_not_autoplace no)
@@
 		)
 		(property "Footprint" ""
-			(at 129.54 95.25 0)
+			(at 139.7 95.25 0)
 			(hide yes)
 			(show_name no)
@@
 		)
 		(property "Datasheet" ""
-			(at 129.54 95.25 0)
+			(at 139.7 95.25 0)
 			(hide yes)
 			(show_name no)
@@
 		)
 		(property "Description" "Power symbol creates a global label with name \"GND\" , ground"
-			(at 129.54 95.25 0)
-			(hide yes)
-			(show_name no)
+			(at 139.7 95.25 0)
+			(hide yes)
+			(show_name no)

Commit message: fc: add footprints
Parts:
- C17, C18: footprint (none) -> Stratus:C_0402
- J1: footprint (none) -> Connector_USB:USB_C_Receptacle_GCT_USB4110
- J2: footprint (none) -> Connector_Card:microSD_HC_Molex_104031-0811
- J4: footprint (none) -> Connector_JST:JST_SH_SM03B-SRSS-TB_1x03-1MP_P1.00mm_Horizontal
- J5: footprint (none) -> Connector_JST:JST_SH_SM02B-SRSS-TB_1x02-1MP_P1.00mm_Horizontal
- J6: footprint (none) -> Connector_JST:JST_SH_SM04B-SRSS-TB_1x04-1MP_P1.00mm_Horizontal
- J7: footprint (none) -> Connector_JST:JST_SH_SM05B-SRSS-TB_1x05-1MP_P1.00mm_Horizontal
- R7, R8: footprint (none) -> Stratus:R_0402
- U5: footprint MICROQFN16_1P25X3P55X0P4_STM -> EMIF06-MSD02N16:EMIF06-MSD02N16
Connections:
- net V_3V3: no longer J2.9 (DET), U5.1 (WD/CD)
- no-connect marks 3 -> 5
Changed lines of the file:
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@@
 	)
 	(junction
-		(at 170.18 73.66)
-		(diameter 0)
-		(color 0 0 0 0)
-	)
-	(junction
 		(at 210.82 76.2)
 		(diameter 0)
@@
 	)
 	(no_connect
+		(at 185.42 44.45)
+	)
+	(no_connect
 		(at 156.21 156.21)
 	)
 	(no_connect
+		(at 156.21 73.66)
+	)
+	(no_connect
 		(at 58.42 78.74)
 	)
@@
 	(wire
 		(pts
-			(xy 170.18 44.45) (xy 170.18 73.66)
-		)
-		(stroke
-			(width 0)
-			(type default)
-		)
-	)
-	(wire
-		(pts
 			(xy 139.7 82.55) (xy 129.54 82.55)
 		)
@@
 	(wire
 		(pts
-			(xy 156.21 73.66) (xy 179.07 73.66)
-		)
-		(stroke
-			(width 0)
-			(type default)
-		)
-	)
-	(wire
-		(pts
 			(xy 110.49 73.66) (xy 113.03 73.66)
 		)
@@
 	(wire
 		(pts
-			(xy 176.53 44.45) (xy 185.42 44.45)
-		)
-		(stroke
-			(width 0)
-			(type default)
-		)
-	)
-	(wire
-		(pts
 			(xy 156.21 53.34) (xy 185.42 53.34)
 		)
@@
 		)
 	)
-	(label "SD_DET"
-		(at 176.53 44.45 0)
-		(effects
-			(font
-				(size 1.27 1.27)
-			)
-			(justify left bottom)
-		)
-	)
 	(label "SD_DAT0"
 		(at 185.42 116.84 180)
@@
 		)
 	)
-	(label "SD_DET"
-		(at 179.07 73.66 180)
-		(effects
-			(font
-				(size 1.27 1.27)
-			)
-			(justify right bottom)
-		)
-	)
 	(label "ESC_M2"
 		(at 130.81 120.65 180)
@@
 		)
 	)
-	(global_label "V_3V3"
-		(shape input)
-		(at 170.18 44.45 90)
-		(fields_autoplaced yes)
-		(effects
-			(font
-				(size 1.27 1.27)
-			)
-			(justify left)
-		)
-		(property "Intersheetrefs" "${INTERSHEET_REFS}"
-			(at 170.18 35.901 90)
-			(hide yes)
-			(show_name no)
-			(do_not_autoplace no)
-			(effects
-				(font
-					(size 1.27 1.27)
-				)
-				(justify left)
-			)
-		)
-	)
 	(global_label "V_5V"
 		(shape input)
@@
 			)
 		)
-		(property "Footprint" ""
+		(property "Footprint" "Stratus:C_0402"
 			(at 129.54 87.63 0)
 			(hide yes)
@@
 			)
 		)
-		(property "Footprint" ""
+		(property "Footprint" "Connector_JST:JST_SH_SM03B-SRSS-TB_1x03-1MP_P1.00mm_Horizontal"
 			(at 120.65 153.67 0)
 			(hide yes)
@@
 			)
 		)
-		(property "Footprint" ""
+		(property "Footprint" "Connector_JST:JST_SH_SM04B-SRSS-TB_1x04-1MP_P1.00mm_Horizontal"
 			(at 151.13 128.27 0)
 			(hide yes)
@@
 			)
 		)
-		(property "Footprint" "MICROQFN16_1P25X3P55X0P4_STM"
+		(property "Footprint" "EMIF06-MSD02N16:EMIF06-MSD02N16"
 			(at 185.42 43.18 0)
 			(hide yes)
@@
 			)
 		)
-		(property "Footprint" ""
+		(property "Footprint" "Connector_USB:USB_C_Receptacle_GCT_USB4110"
 			(at 46.99 66.04 0)
 			(hide yes)
@@
 			)
 		)
-		(property "Footprint" ""
+		(property "Footprint" "Stratus:R_0402"
 			(at 63.5 55.88 0)
 			(hide yes)
@@
 			)
 		)
-		(property "Footprint" ""
+		(property "Footprint" "Connector_Card:microSD_HC_Molex_104031-0811"
 			(at 81.28 43.18 0)
 			(hide yes)
@@
 			)
 		)
-		(property "Footprint" ""
+		(property "Footprint" "Stratus:R_0402"
 			(at 63.5 58.42 0)
 			(hide yes)
@@
 			)
 		)
-		(property "Footprint" ""
+		(property "Footprint" "Connector_JST:JST_SH_SM05B-SRSS-TB_1x05-1MP_P1.00mm_Horizontal"
 			(at 151.13 158.75 0)
 			(hide yes)
@@
 			)
 		)
-		(property "Footprint" ""
+		(property "Footprint" "Connector_JST:JST_SH_SM02B-SRSS-TB_1x02-1MP_P1.00mm_Horizontal"
 			(at 120.65 167.64 0)
 			(hide yes)
@@
 			)
 		)
-		(property "Footprint" ""
+		(property "Footprint" "Stratus:C_0402"
 			(at 139.7 87.63 0)
 			(hide yes)

Commit message: fc: fix peripherals
Connections:
- net SD_DAT1: no longer names the net of U5.9 (DAT1_EX)
- net SD_DAT2: no longer names the net of U5.14 (DAT2_EX)
- no-connect marks 5 -> 7
Changed lines of the file:
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@@
+	)
+	(no_connect
+		(at 245.11 50.8)
+	)
+	(no_connect
+		(at 245.11 63.5)
 	)
 	(no_connect
@@
 	)
 	(bus_entry
-		(at 186.69 127)
+		(at 187.96 124.46)
 		(size 2.54 2.54)
 		(stroke
@@
 	)
 	(bus_entry
-		(at 186.69 134.62)
+		(at 187.96 132.08)
 		(size 2.54 2.54)
 		(stroke
@@
 	)
 	(bus_entry
-		(at 186.69 129.54)
+		(at 187.96 127)
 		(size 2.54 2.54)
 		(stroke
@@
 	)
 	(bus_entry
-		(at 187.96 119.38)
-		(size 2.54 2.54)
-		(stroke
-			(width 0)
-			(type default)
-		)
-	)
-	(bus_entry
-		(at 186.69 124.46)
+		(at 187.96 121.92)
 		(size 2.54 2.54)
 		(stroke
@@
 	)
 	(bus_entry
-		(at 186.69 132.08)
+		(at 187.96 129.54)
 		(size 2.54 2.54)
 		(stroke
@@
 		)
 	)
-	(bus_entry
-		(at 187.96 106.68)
-		(size 2.54 2.54)
-		(stroke
-			(width 0)
-			(type default)
-		)
-	)
 	(wire
 		(pts
@@
 	(bus
 		(pts
-			(xy 189.23 137.16) (xy 195.58 137.16)
+			(xy 190.5 134.62) (xy 196.85 134.62)
 		)
 		(stroke
@@
 	(wire
 		(pts
-			(xy 185.42 119.38) (xy 187.96 119.38)
-		)
-		(stroke
-			(width 0)
-			(type default)
-		)
-	)
-	(wire
-		(pts
 			(xy 156.21 66.04) (xy 180.34 66.04)
 		)
@@
 	(bus
 		(pts
-			(xy 190.5 109.22) (xy 190.5 121.92)
+			(xy 190.5 109.22) (xy 190.5 119.38)
 		)
 		(stroke
@@
 	(wire
 		(pts
-			(xy 184.15 124.46) (xy 186.69 124.46)
+			(xy 185.42 121.92) (xy 187.96 121.92)
 		)
 		(stroke
@@
 	(wire
 		(pts
-			(xy 185.42 106.68) (xy 187.96 106.68)
-		)
-		(stroke
-			(width 0)
-			(type default)
-		)
-	)
-	(wire
-		(pts
-			(xy 184.15 129.54) (xy 186.69 129.54)
+			(xy 185.42 127) (xy 187.96 127)
 		)
 		(stroke
@@
 	(wire
 		(pts
-			(xy 184.15 127) (xy 186.69 127)
+			(xy 185.42 124.46) (xy 187.96 124.46)
 		)
 		(stroke
@@
 	(wire
 		(pts
-			(xy 184.15 132.08) (xy 186.69 132.08)
+			(xy 185.42 129.54) (xy 187.96 129.54)
 		)
 		(stroke
@@
 	(bus
 		(pts
-			(xy 190.5 121.92) (xy 196.85 121.92)
+			(xy 190.5 119.38) (xy 196.85 119.38)
 		)
 		(stroke
@@
 	(bus
 		(pts
-			(xy 189.23 127) (xy 189.23 137.16)
-		)
-		(stroke
-			(width 0)
-			(type default)
-		)
-	)
-	(wire
-		(pts
-			(xy 184.15 134.62) (xy 186.69 134.62)
+			(xy 190.5 124.46) (xy 190.5 134.62)
+		)
+		(stroke
+			(width 0)
+			(type default)
+		)
+	)
+	(wire
+		(pts
+			(xy 185.42 132.08) (xy 187.96 132.08)
 		)
 		(stroke
@@
 		)
 	)
-	(label "SD_DAT2"
-		(at 185.42 106.68 180)
-		(effects
-			(font
-				(size 1.27 1.27)
-			)
-			(justify right bottom)
-		)
-	)
 	(label "SD_CMD"
 		(at 245.11 55.88 180)
@@
 	)
 	(label "ESC_M1"
-		(at 184.15 132.08 180)
+		(at 185.42 129.54 180)
 		(effects
 			(font
@@
 	)
 	(label "ESC_M4"
-		(at 184.15 124.46 180)
+		(at 185.42 121.92 180)
 		(effects
 			(font
@@
 	)
 	(label "ESC_TEL"
-		(at 184.15 134.62 180)
+		(at 185.42 132.08 180)
 		(effects
 			(font
@@
 	)
 	(label "ESC_M3"
-		(at 184.15 127 180)
-		(effects
-			(font
-				(size 1.27 1.27)
-			)
-			(justify right bottom)
-		)
-	)
-	(label "SD_DAT1"
-		(at 245.11 63.5 180)
-		(effects
-			(font
-				(size 1.27 1.27)
-			)
-			(justify right bottom)
-		)
-	)
-	(label "SD_DAT1"
-		(at 185.42 119.38 180)
+		(at 185.42 124.46 180)
 		(effects
 			(font
@@
 	)
 	(label "ESC_M2"
-		(at 184.15 129.54 180)
-		(effects
-			(font
-				(size 1.27 1.27)
-			)
-			(justify right bottom)
-		)
-	)
-	(label "SD_DAT2"
-		(at 245.11 50.8 180)
+		(at 185.42 127 180)
 		(effects
 			(font
@@
 	(hierarchical_label "ESC{M[1..4] TEL}"
 		(shape bidirectional)
-		(at 195.58 137.16 0)
+		(at 196.85 134.62 0)
 		(effects
 			(font
@@
 		)
 	)
-	(hierarchical_label "SD{DAT[0..3] CMD CLK}"
+	(hierarchical_label "SD{DAT0 DAT3 CMD CLK}"
 		(shape bidirectional)
-		(at 196.85 121.92 0)
-		(effects
-			(font
+		(at 196.85 119.38 0)
+		(effects
+			(font

Commit message: fc: schematic tweaks; prelim power stage + connector layout
Parts:
- J2: footprint Connector_Card:microSD_HC_Molex_104031-0811 -> Stratus:0473092651
- U5: footprint EMIF06-MSD02N16:EMIF06-MSD02N16 -> Stratus:EMIF06-MSD02N16
Connections:
- net at U5.3 (DAT2_IN): no longer J2.1 (DAT2)
- net at U5.8 (DAT1_IN): no longer J2.8 (DAT1)
- no-connect marks 7 -> 11
Changed lines of the file:
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@@
+	)
+	(no_connect
+		(at 185.42 50.8)
 	)
 	(no_connect
@@
 	)
 	(no_connect
+		(at 156.21 68.58)
+	)
+	(no_connect
 		(at 245.11 63.5)
 	)
@@
 	)
 	(no_connect
+		(at 185.42 63.5)
+	)
+	(no_connect
 		(at 58.42 78.74)
+	)
+	(no_connect
+		(at 156.21 50.8)
 	)
 	(bus_entry
@@
 	(wire
 		(pts
-			(xy 156.21 50.8) (xy 185.42 50.8)
-		)
-		(stroke
-			(width 0)
-			(type default)
-		)
-	)
-	(wire
-		(pts
 			(xy 58.42 58.42) (xy 60.96 58.42)
 		)
@@
 	(wire
 		(pts
-			(xy 182.88 63.5) (xy 182.88 68.58)
-		)
-		(stroke
-			(width 0)
-			(type default)
-		)
-	)
-	(wire
-		(pts
 			(xy 60.96 71.12) (xy 58.42 71.12)
 		)
@@
 	(wire
 		(pts
-			(xy 185.42 63.5) (xy 182.88 63.5)
-		)
-		(stroke
-			(width 0)
-			(type default)
-		)
-	)
-	(wire
-		(pts
 			(xy 185.42 127) (xy 187.96 127)
 		)
@@
 		(pts
 			(xy 127 82.55) (xy 129.54 82.55)
-		)
-		(stroke
-			(width 0)
-			(type default)
-		)
-	)
-	(wire
-		(pts
-			(xy 156.21 68.58) (xy 182.88 68.58)
 		)
 		(stroke
@@
 			)
 		)
-		(property "Footprint" "EMIF06-MSD02N16:EMIF06-MSD02N16"
+		(property "Footprint" "Stratus:EMIF06-MSD02N16"
 			(at 185.42 43.18 0)
 			(hide yes)
@@
 			)
 		)
-		(property "Footprint" "Connector_Card:microSD_HC_Molex_104031-0811"
+		(property "Footprint" "Stratus:0473092651"
 			(at 81.28 43.18 0)
 			(hide yes)

Commit message: fc: schematic footprint changes
Connections:
- net at U5.3 (DAT2_IN): now also J2.1 (DAT2)
- net at U5.8 (DAT1_IN): now also J2.8 (DAT1)
- no-connect marks 11 -> 7
Changed lines of the file:
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@@
-	)
-	(no_connect
-		(at 185.42 50.8)
 	)
 	(no_connect
@@
 	)
 	(no_connect
-		(at 156.21 68.58)
-	)
-	(no_connect
 		(at 245.11 63.5)
 	)
@@
 	)
 	(no_connect
-		(at 185.42 63.5)
-	)
-	(no_connect
 		(at 58.42 78.74)
 	)
-	(no_connect
-		(at 156.21 50.8)
-	)
 	(bus_entry
 		(at 187.96 124.46)
@@
 	(wire
 		(pts
+			(xy 156.21 50.8) (xy 185.42 50.8)
+		)
+		(stroke
+			(width 0)
+			(type default)
+		)
+	)
+	(wire
+		(pts
 			(xy 58.42 58.42) (xy 60.96 58.42)
 		)
@@
 	(wire
 		(pts
+			(xy 182.88 63.5) (xy 182.88 68.58)
+		)
+		(stroke
+			(width 0)
+			(type default)
+		)
+	)
+	(wire
+		(pts
 			(xy 60.96 71.12) (xy 58.42 71.12)
 		)
@@
 	(wire
 		(pts
+			(xy 185.42 63.5) (xy 182.88 63.5)
+		)
+		(stroke
+			(width 0)
+			(type default)
+		)
+	)
+	(wire
+		(pts
 			(xy 185.42 127) (xy 187.96 127)
 		)
@@
 		)
 		(stroke
+			(width 0)
+			(type default)
+		)
+	)
+	(wire
+		(pts
+			(xy 156.21 68.58) (xy 182.88 68.58)
+		)
+		(stroke

Commit message: fc: PDN; further layout work
Connections:
- net ESC_M1 renamed ESC.M1
- net ESC_M2 renamed ESC.M2
- net ESC_M3 renamed ESC.M3
- net ESC_M4 renamed ESC.M4
- net ESC_TEL renamed ESC.TEL
- net SD_CLK renamed SD.CLK
- net SD_CMD renamed SD.CMD
- net SD_DAT0 renamed SD.DAT0
- net SD_DAT3 renamed SD.DAT3
Changed lines of the file:
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@@
 		)
 	)
-	(label "SD_DAT3"
+	(label "SD.DAT3"
 		(at 245.11 53.34 180)
 		(effects
@@
 		)
 	)
-	(label "ESC_TEL"
+	(label "ESC.TEL"
 		(at 130.81 128.27 180)
 		(effects
@@
 		)
 	)
-	(label "SD_CMD"
+	(label "SD.CMD"
 		(at 245.11 55.88 180)
 		(effects
@@
 		)
 	)
-	(label "ESC_M1"
+	(label "ESC.M1"
 		(at 185.42 129.54 180)
 		(effects
@@
 		)
 	)
-	(label "ESC_M4"
+	(label "ESC.M4"
 		(at 185.42 121.92 180)
 		(effects
@@
 		)
 	)
-	(label "ESC_M4"
+	(label "ESC.M4"
 		(at 130.81 115.57 180)
 		(effects
@@
 		)
 	)
-	(label "SD_DAT0"
+	(label "SD.DAT0"
 		(at 185.42 116.84 180)
 		(effects
@@
 		)
 	)
-	(label "ESC_M3"
+	(label "ESC.M3"
 		(at 130.81 118.11 180)
 		(effects
@@
 		)
 	)
-	(label "SD_DAT0"
+	(label "SD.DAT0"
 		(at 245.11 60.96 180)
 		(effects
@@
 		)
 	)
-	(label "ESC_M1"
+	(label "ESC.M1"
 		(at 130.81 123.19 180)
 		(effects
@@
 		)
 	)
-	(label "SD_CLK"
+	(label "SD.CLK"
 		(at 185.42 114.3 180)
 		(effects
@@
 		)
 	)
-	(label "ESC_M2"
+	(label "ESC.M2"
 		(at 130.81 120.65 180)
 		(effects
@@
 		)
 	)
-	(label "ESC_TEL"
+	(label "ESC.TEL"
 		(at 185.42 132.08 180)
 		(effects
@@
 		)
 	)
-	(label "ESC_M3"
+	(label "ESC.M3"
 		(at 185.42 124.46 180)
 		(effects
@@
 		)
 	)
-	(label "SD_DAT3"
+	(label "SD.DAT3"
 		(at 185.42 109.22 180)
 		(effects
@@
 		)
 	)
-	(label "SD_CMD"
+	(label "SD.CMD"
 		(at 185.42 111.76 180)
 		(effects
@@
 		)
 	)
-	(label "ESC_M2"
+	(label "ESC.M2"
 		(at 185.42 127 180)
 		(effects
@@
 		)
 	)
-	(label "SD_CLK"
+	(label "SD.CLK"
 		(at 245.11 58.42 180)
 		(effects

Commit message: fc: routing and pours
Connections:
- net at U5.3 (DAT2_IN): no longer J2.1 (DAT2)
- net at U5.8 (DAT1_IN): no longer J2.8 (DAT1)
- no-connect marks 7 -> 11
Changed lines of the file:
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@@
+	)
+	(no_connect
+		(at 156.21 68.58)
+	)
+	(no_connect
+		(at 185.42 50.8)
 	)
 	(no_connect
@@
 	)
 	(no_connect
+		(at 156.21 50.8)
+	)
+	(no_connect
 		(at 156.21 156.21)
 	)
@@
 	)
 	(no_connect
+		(at 185.42 63.5)
+	)
+	(no_connect
 		(at 245.11 63.5)
 	)
@@
 	(wire
 		(pts
-			(xy 156.21 50.8) (xy 185.42 50.8)
-		)
-		(stroke
-			(width 0)
-			(type default)
-		)
-	)
-	(wire
-		(pts
 			(xy 58.42 58.42) (xy 60.96 58.42)
 		)
@@
 	(wire
 		(pts
-			(xy 182.88 63.5) (xy 182.88 68.58)
-		)
-		(stroke
-			(width 0)
-			(type default)
-		)
-	)
-	(wire
-		(pts
 			(xy 60.96 71.12) (xy 58.42 71.12)
 		)
@@
 	(wire
 		(pts
-			(xy 185.42 63.5) (xy 182.88 63.5)
-		)
-		(stroke
-			(width 0)
-			(type default)
-		)
-	)
-	(wire
-		(pts
 			(xy 185.42 127) (xy 187.96 127)
 		)
@@
 		)
 		(stroke
-			(width 0)
-			(type default)
-		)
-	)
-	(wire
-		(pts
-			(xy 156.21 68.58) (xy 182.88 68.58)
-		)
-		(stroke
