File: hardware/fc/peripherals.kicad_sch (KiCad schematic)
At the start: 13 parts, among them J1 USB4110-GF-A, J2 Micro_SD_Card_Det1, J3 FROM_ESC, J4 CAM, J5 CAM_CC, J6 ELRS, J7 VTX, U4 USBLC6-2SC6, U5 EMIF06-MSD02N16

Commit message: fc: footprints
Parts:
- U4: footprint Package_TO_SOT_SMD:SOT-23-6 -> Stratus:USBLC6-2SC6
Changed lines of the file:
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@@
 			)
 		)
-		(property "Footprint" "Package_TO_SOT_SMD:SOT-23-6"
+		(property "Footprint" "Stratus:USBLC6-2SC6"
 			(at 81.28 72.39 0)
 			(hide yes)
