File: hardware/fc/power.kicad_sch (KiCad schematic)
At the start: 30 parts, among them U1 TPS7A8101DRBR, U10 TPS2116DRL, U2 TPS7A8101DRBR, U3 LMR51420YFDDCR

Commit message: fc: schematic tweaks; prelim power stage + connector layout
Connections:
- net GND: now also U10.4 (PR1), U10.5 (MODE)
- net V_BUS: no longer U10.4 (PR1), U10.5 (MODE)
Other:
- note added: "To RP2354A"
- note removed: "To RP2354B"
- moved on the sheet: C29, C30, C31, U10

Commit message: fc: schematic footprint changes
Connections:
- net GND: no longer U10.4 (PR1), U10.5 (MODE)
- net V_BUS: now also U10.4 (PR1), U10.5 (MODE)
Other:
- note added: "To RP2354B"
- note removed: "To RP2354A"
- moved on the sheet: C29, C30, C31, U10

Commit message: fc: add power pours
Connections:
- net GND: now also U10.4 (PR1), U10.5 (MODE)
- net V_BUS: no longer U10.4 (PR1), U10.5 (MODE)
Other:
- note added: "To RP2354B + OSD"
- note removed: "To RP2354B"
- moved on the sheet: C29, C30, C31, U10

Commit message: fc: footprints
Parts:
- U1, U2: footprint Package_SON:VSON-8-1EP_3x3mm_P0.65mm_EP1.65x2.4mm -> Stratus:TPS7A8101DRBR
- U10: footprint Package_TO_SOT_SMD:SOT-583-8 -> Stratus:TPS2116DRL
Changed lines of the file:
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@@
 			)
 		)
-		(property "Footprint" "Package_TO_SOT_SMD:SOT-583-8"
+		(property "Footprint" "Stratus:TPS2116DRL"
 			(at 212.09 89.662 0)
 			(hide yes)
@@
 			)
 		)
-		(property "Footprint" "Package_SON:VSON-8-1EP_3x3mm_P0.65mm_EP1.65x2.4mm"
+		(property "Footprint" "Stratus:TPS7A8101DRBR"
 			(at 130.81 114.3 0)
 			(hide yes)
@@
 			)
 		)
-		(property "Footprint" "Package_SON:VSON-8-1EP_3x3mm_P0.65mm_EP1.65x2.4mm"
+		(property "Footprint" "Stratus:TPS7A8101DRBR"
 			(at 238.76 114.3 0)
 			(hide yes)
