File: hardware/fc/fc.kicad_pcb (KiCad board)
At the start: 6 copper layers, 35 x 35 mm, 108 parts, among them J1 USB4110-GF-A, J2 Micro_SD_Card_Det1, J3 FROM_ESC, J4 CAM, J5 CAM_CC, J6 ELRS, J7 VTX, SW1 Push, U1 TPS7A8101DRBR, U10 TPS2116DRL, U11 OPA354AIDBVR, U12 RP2354A, U2 TPS7A8101DRBR, U3 LMR51420YFDDCR, U4 USBLC6-2SC6, U5 EMIF06-MSD02N16, U6 LSM6DSK320X, U8 TS5A3159ADCK, U9 LMV7219M7X, X1 ABM8-272-T3

Commit message: fc: edit values to add temperature drift robustness to OSD
Parts:
- C27: value 1uF -> 0.1uF
- R28: value 100k -> 1M
- R30: value 1.2k -> 1k
Changed lines of the file:
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@@
 			)
 		)
-		(property "Value" "100k"
+		(property "Value" "1M"
 			(at 0 -1.17 0)
 			(layer "B.Fab")
@@
 			)
 		)
-		(property "Value" "1.2k"
+		(property "Value" "1k"
 			(at 0 -1.17 90)
 			(layer "B.Fab")
@@
 			)
 		)
-		(property "Value" "1uF"
+		(property "Value" "0.1uF"
 			(at 0 -1.17 0)
 			(layer "B.Fab")
@@
 	)
 	(segment
+		(start 163.6025 119.727499)
+		(end 164.429999 118.9)
+		(width 0.15)
+		(layer "B.Cu")
+		(net "Net-(U9-+)")
+	)
+	(segment
+		(start 165.370001 118.9)
+		(end 164.429999 118.9)
+		(width 0.15)
+		(layer "B.Cu")
+		(net "Net-(U9-+)")
+	)
+	(segment
+		(start 163.6025 119.86)
+		(end 163.6025 119.727499)
+		(width 0.15)
+		(layer "B.Cu")
+		(net "Net-(U9-+)")
+	)
+	(segment
 		(start 162.479998 117.909999)
 		(end 162.299999 117.73)
@@
 		(net "Net-(R10-Pad1)")
 	)
-	(segment
-		(start 163.6025 119.727499)
-		(end 164.429999 118.9)
-		(width 0.15)
-		(layer "B.Cu")
-		(net "Net-(U9-+)")
-	)
-	(segment
-		(start 165.370001 118.9)
-		(end 164.429999 118.9)
-		(width 0.15)
-		(layer "B.Cu")
-		(net "Net-(U9-+)")
-	)
-	(segment
-		(start 163.6025 119.86)
-		(end 163.6025 119.727499)
-		(width 0.15)
-		(layer "B.Cu")
-		(net "Net-(U9-+)")
-	)
 	(zone
 		(net "V_BAT")
@@
 			)
 		)
-	)
-	(zone
-		(layer "B.Cu")
-		(hatch edge 0.5)
-		(connect_pads
-			(clearance 0)
-		)
-		(min_thickness 0.25)
-		(keepout
-			(tracks allowed)
-			(vias allowed)
-			(pads allowed)
-			(copperpour allowed)
-			(footprints not_allowed)
-		)
-		(placement
-			(enabled no)
-			(sheetname "/")
-		)
-		(fill
-			(thermal_gap 0.5)
-			(thermal_bridge_width 0.5)
-			(island_removal_mode 0)
-		)
-		(polygon
-			(pts
-				(xy 145.5 99.6175) (xy 157.5 99.6175) (xy 157.5 111.9775) (xy 145.5 111.9775)
-			)
-		)

Commit message: fc: final resistor edit
Parts:
- R28: value 1M -> 220k
Changed lines of the file:
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@@
 			)
 		)
-		(property "Value" "1M"
+		(property "Value" "220k"
 			(at 0 -1.17 0)
 			(layer "B.Fab")
