File: hardware/fc/fc.kicad_sch (KiCad schematic)
At the start: 40 parts, among them SW1 Push, U12 RP2354A, X1 ABM8-272-T3

Commit message: fc: meta
Other:
- title: RP2354B; ICM-40609-D Flight Controller -> RP2354B; LSM6DSK320X Flight Controller
Changed lines of the file:
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@@
 	(paper "A4")
 	(title_block
-		(title "RP2354B; ICM-40609-D Flight Controller")
+		(title "RP2354B; LSM6DSK320X Flight Controller")
 		(date "2026-09-17")
 		(rev "1")
